File: KiCAD/8-buttons.kicad_sch (KiCad schematic)
At the start: 19 parts, among them U1 74HC165, U2 TLC5916

Commit message: fix DRC errors
Changed lines of the file:
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@@
-	)
-	(junction
-		(at 166.37 57.15)
-		(diameter 0)
-		(color 0 0 0 0)
 	)
 	(junction
@@
 		(color 0 0 0 0)
 	)
-	(junction
-		(at 205.74 57.15)
-		(diameter 0)
-		(color 0 0 0 0)
-	)
-	(junction
-		(at 245.11 57.15)
-		(diameter 0)
-		(color 0 0 0 0)
-	)
 	(no_connect
 		(at 248.92 109.22)
@@
 	(wire
 		(pts
-			(xy 205.74 45.72) (xy 205.74 57.15)
-		)
-		(stroke
-			(width 0)
-			(type default)
-		)
-	)
-	(wire
-		(pts
 			(xy 69.85 115.57) (xy 69.85 116.84)
 		)
@@
 	(wire
 		(pts
-			(xy 245.11 43.18) (xy 245.11 57.15)
-		)
-		(stroke
-			(width 0)
-			(type default)
-		)
-	)
-	(wire
-		(pts
 			(xy 248.92 81.28) (xy 248.92 69.85)
 		)
@@
 		)
 		(stroke
-			(width 0)
-			(type default)
-		)
-	)
-	(wire
-		(pts
-			(xy 166.37 48.26) (xy 166.37 57.15)
-		)
-		(stroke
