File: KiCAD/DrumKitButtons.kicad_pcb (KiCad board)
At the start: 2 copper layers, 318 x 28 mm, 44 parts, among them J1 Input, J2 Output, U1 74HC165, U2 TLC5916, U3 74HC165, U4 TLC5916

Commit message: fix DRC errors
Parts:
- moved R3 224.8 mm to (355.1, 90.7)
- moved R17 209.7 mm to (130.3, 90.6)
- moved R2 202.4 mm to (295.0, 90.6), turned to 0 degrees
- moved R5 179.7 mm to (339.9, 90.7)
- moved R15 165.2 mm to (145.1, 90.7)
- moved R18 165.0 mm to (190.1, 90.7)
- moved R7 149.9 mm to (325.3, 90.7)
- moved R10 142.7 mm to (92.7, 83.8), turned to -90 degrees
- moved R4 135.3 mm to (280.3, 90.7)
- moved R13 120.1 mm to (160.2, 90.7)
- moved R16 120.1 mm to (205.2, 90.7)
- moved R9 90.4 mm to (310.3, 90.7)
- moved R14 75.1 mm to (219.9, 90.7)
- moved R6 75.1 mm to (265.2, 90.6)
- moved R11 74.9 mm to (175.3, 90.6)
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Connections:
- J1 pad 4: /DI_{LED} -> /DO_{LED}
- J1 pad 5: /DO_{SW} -> /DI_{SW}
- J2 pad 4: /DO_{LED} -> /DI_{LED}
- J2 pad 5: /DI_{SW} -> /DO_{SW}
Routing:
- net (no net): track 690.1 -> 0.00 mm
- net /Button Bank 0/SW_{0}: track 0.00 -> 235.9 mm
- net /Button Bank 0/LED_{5}: track 0.00 -> 234.1 mm
- net /Button Bank 0/LED_{6}: track 0.00 -> 220.8 mm
- net /Button Bank 0/SW_{4}: track 66.9 -> 287.5 mm
- net /Button Bank 1/LED_{2}: track 256.1 -> 40.7 mm
- net /Button Bank 0/LED_{0}: track 0.00 -> 195.9 mm
- net /Button Bank 0/LED_{1}: track 0.00 -> 178.1 mm
- net /Button Bank 1/LED_{3}: track 161.7 -> 22.2 mm
- net /Button Bank 1/LED_{6}: track 234.1 -> 103.9 mm
- net /Button Bank 1/LED_{7}: track 220.8 -> 92.3 mm
- net /Button Bank 1/SW_{2}: track 218.1 -> 90.2 mm, vias 0 -> 1
- net /Button Bank 1/SW_{1}: track 235.9 -> 108.1 mm
- net /Button Bank 1/SW_{3}: track 200.6 -> 73.4 mm
- net /Button Bank 1/SW_{0}: track 0.00 -> 124.8 mm, vias 0 -> 1
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Other:
- board size 318 x 28 mm -> 318 x 28.6 mm
- board text added: "https://github.com/aseanwatson/DrumKitButtons/releases/tag/${REV}"
- board text removed: "https://github.com/aseanwatson/DrumKitButtons/releases/tag/v2"

Commit message: elimiate vias
Parts:
- moved R18 120.2 mm to (310.3, 90.7)
- moved R9 120.2 mm to (190.1, 90.7)
- moved R13 120.1 mm to (280.3, 90.7)
- moved R4 120.1 mm to (160.2, 90.7)
- moved R16 120.1 mm to (325.3, 90.7)
- moved R7 120.1 mm to (205.2, 90.7)
- moved R15 120.1 mm to (265.2, 90.6)
- moved R6 120.1 mm to (145.1, 90.7)
- moved R14 120.0 mm to (339.9, 90.7)
- moved R5 120.0 mm to (219.9, 90.7)
- moved SW1 120.0 mm to (175.8, 81.0)
- moved SW10 120.0 mm to (355.8, 81.0)
- moved SW11 120.0 mm to (280.8, 81.0)
- moved SW12 120.0 mm to (340.8, 81.0)
- moved SW13 120.0 mm to (265.8, 81.0)
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Routing:
- net /Button Bank 1/LED_{2}: track 40.7 -> 161.7 mm
- net /Button Bank 0/LED_{2}: track 161.7 -> 40.7 mm
- net /Button Bank 1/LED_{3}: track 22.2 -> 142.7 mm
- net /Button Bank 0/LED_{3}: track 142.7 -> 22.2 mm
- net /Button Bank 1/LED_{0}: track 78.0 -> 195.9 mm
- net /Button Bank 0/LED_{0}: track 195.9 -> 78.0 mm
- net /Button Bank 1/LED_{1}: track 60.9 -> 178.1 mm
- net /Button Bank 0/LED_{1}: track 178.1 -> 60.9 mm
- net /Button Bank 1/LED_{4}: track 128.7 -> 245.8 mm
- net /Button Bank 0/LED_{4}: track 245.8 -> 128.7 mm
- net /Button Bank 1/LED_{6}: track 103.9 -> 220.8 mm
- net /Button Bank 0/LED_{6}: track 220.8 -> 103.9 mm
- net /Button Bank 1/LED_{7}: track 92.3 -> 209.2 mm
- net /Button Bank 0/LED_{7}: track 209.2 -> 92.3 mm
- net /Button Bank 1/LED_{5}: track 117.4 -> 234.1 mm
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Other:
- board size 318 x 28.6 mm -> 316.6 x 28.5 mm
- board text removed: "0"
- board text removed: "1"
- board text removed: "10"
- board text removed: "11"
- board text removed: "12"
- board text removed: "13"
- board text removed: "14"
- board text removed: "15"
- board text removed: "2"
- board text removed: "3"
- board text removed: "4"
- board text removed: "5"
- board text removed: "6"
- board text removed: "7"
- board text removed: "8"
- board text removed: "9"
