File: KiCAD/DrumKitButtons.kicad_pcb (KiCad board)
At the start: 2 copper layers, 316.6 x 28.5 mm, 44 parts, among them J1 Input, J2 Output, U1 74HC165, U2 TLC5916, U3 74HC165, U4 TLC5916

Commit message: reorder buttons/leds
Parts:
- J1: value Input -> Output
- J2: value Output -> Input
- R1: renamed from R18; value 47R -> 400R
- R11: renamed from R10; value 400R -> 47R
- R2: renamed from R9; value 47R -> 400R
- R3: renamed from R1; value 400R -> 47R
- moved R1 218.3 mm to (92.7, 73.7), turned to -90 degrees
- moved R11 158.4 mm to (250.2, 90.6), turned to 0 degrees
- moved R10 105.0 mm to (235.3, 90.6)
- moved R18 104.9 mm to (355.1, 90.7)
- moved R2 97.6 mm to (92.7, 83.8), turned to -90 degrees
- moved SW14 90.0 mm to (340.8, 81.0)
- moved SW1 90.0 mm to (145.8, 81.0)
- moved SW6 90.0 mm to (220.8, 81.0)
- moved SW9 90.0 mm to (265.8, 81.0)
- moved R5 75.1 mm to (160.2, 90.7)
- moved R13 74.7 mm to (280.3, 90.7)
- moved R16 60.1 mm to (325.3, 90.7)
- moved R8 60.1 mm to (205.2, 90.7)
- moved SW8 45.0 mm to (250.8, 81.0)
- moved SW0 45.0 mm to (130.8, 81.0)
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- renumbered H4 to H3, H3 to H4, R8 to R10, R11 to R12, R12 to R13, R13 to R14, R14 to R15, R15 to R16, R16 to R17, R17 to R18, R2 to R4, R3 to R5, R5 to R6, R4 to R7, R6 to R8, R7 to R9, SW1 to SW0, SW2 to SW1, SW11 to SW10, SW12 to SW11, SW13 to SW12, SW14 to SW13, SW15 to SW14, SW16 to SW15, SW3 to SW2, SW4 to SW3, SW5 to SW4, SW6 to SW5, SW7 to SW6, SW8 to SW7, SW9 to SW8, SW10 to SW9, U4 to U2, U2 to U4
Connections:
- J1 pad 4: /DO_{LED} -> /DI_{LED}
- J1 pad 5: /DI_{SW} -> /DO_{SW}
- J2 pad 4: /DI_{LED} -> /DO_{LED}
- J2 pad 5: /DO_{SW} -> /DI_{SW}
- R1 pad 1: /Button Bank 1/SW_{7} -> /Button Bank 1/Net-(U2-R-EXT)
- R10 pad 1: /Button Bank 0/SW_{3} -> /Button Bank 0/SW_{7}
- R11 pad 1: Net-(U4-R-EXT) -> /Button Bank 1/SW_{0}
- R12 pad 1: /Button Bank 1/SW_{0} -> /Button Bank 1/SW_{1}
- R13 pad 1: /Button Bank 1/SW_{4} -> /Button Bank 1/SW_{2}
- R14 pad 1: /Button Bank 1/SW_{1} -> /Button Bank 1/SW_{3}
- R15 pad 1: /Button Bank 1/SW_{5} -> /Button Bank 1/SW_{4}
- R16 pad 1: /Button Bank 1/SW_{2} -> /Button Bank 1/SW_{5}
- R18 pad 1: /Button Bank 1/SW_{3} -> /Button Bank 1/SW_{7}
- R2 pad 1: /Button Bank 0/SW_{7} -> /Button Bank 0/Net-(U2-R-EXT)
- R3 pad 1: Net-(U2-R-EXT) -> /Button Bank 0/SW_{0}
- R4 pad 1: /Button Bank 0/SW_{0} -> /Button Bank 0/SW_{1}
- R5 pad 1: /Button Bank 0/SW_{4} -> /Button Bank 0/SW_{2}
- R6 pad 1: /Button Bank 0/SW_{5} -> /Button Bank 0/SW_{4}
- R7 pad 1: /Button Bank 0/SW_{1} -> /Button Bank 0/SW_{3}
- R8 pad 1: /Button Bank 0/SW_{2} -> /Button Bank 0/SW_{5}
- SW1 pad 2: /Button Bank 0/SW_{4} -> /Button Bank 0/SW_{1}
- SW1 pad 6: /Button Bank 0/LED_{4} -> /Button Bank 0/LED_{1}
- SW10 pad 2: /Button Bank 1/SW_{1} -> /Button Bank 1/SW_{2}
- SW10 pad 6: /Button Bank 1/LED_{1} -> /Button Bank 1/LED_{2}
- SW11 pad 2: /Button Bank 1/SW_{5} -> /Button Bank 1/SW_{3}
- SW11 pad 6: /Button Bank 1/LED_{5} -> /Button Bank 1/LED_{3}
- SW12 pad 2: /Button Bank 1/SW_{2} -> /Button Bank 1/SW_{4}
- SW12 pad 6: /Button Bank 1/LED_{2} -> /Button Bank 1/LED_{4}
- SW13 pad 2: /Button Bank 1/SW_{6} -> /Button Bank 1/SW_{5}
- SW13 pad 6: /Button Bank 1/LED_{6} -> /Button Bank 1/LED_{5}
- SW14 pad 2: /Button Bank 1/SW_{3} -> /Button Bank 1/SW_{6}
- SW14 pad 6: /Button Bank 1/LED_{3} -> /Button Bank 1/LED_{6}
- SW2 pad 2: /Button Bank 0/SW_{1} -> /Button Bank 0/SW_{2}
- SW2 pad 6: /Button Bank 0/LED_{1} -> /Button Bank 0/LED_{2}
- SW3 pad 2: /Button Bank 0/SW_{5} -> /Button Bank 0/SW_{3}
- SW3 pad 6: /Button Bank 0/LED_{5} -> /Button Bank 0/LED_{3}
- SW4 pad 2: /Button Bank 0/SW_{2} -> /Button Bank 0/SW_{4}
- SW4 pad 6: /Button Bank 0/LED_{2} -> /Button Bank 0/LED_{4}
- SW5 pad 2: /Button Bank 0/SW_{6} -> /Button Bank 0/SW_{5}
- SW5 pad 6: /Button Bank 0/LED_{6} -> /Button Bank 0/LED_{5}
- SW6 pad 2: /Button Bank 0/SW_{3} -> /Button Bank 0/SW_{6}
- SW6 pad 6: /Button Bank 0/LED_{3} -> /Button Bank 0/LED_{6}
- SW9 pad 2: /Button Bank 1/SW_{4} -> /Button Bank 1/SW_{1}
- SW9 pad 6: /Button Bank 1/LED_{4} -> /Button Bank 1/LED_{1}
- U2 pad 15: Net-(U4-R-EXT) -> /Button Bank 1/Net-(U2-R-EXT)
- U4 pad 15: Net-(U2-R-EXT) -> /Button Bank 0/Net-(U2-R-EXT)
Routing:
- net /Button Bank 0/SW_{1}: track 105.9 -> 165.0 mm
- net /Button Bank 1/SW_{5}: track 274.6 -> 331.4 mm
- net /Button Bank 0/SW_{5}: track 162.0 -> 217.7 mm
- net /Button Bank 1/SW_{3}: track 183.4 -> 235.9 mm
- net /Button Bank 0/LED_{1}: track 58.5 -> 109.9 mm
- net /Button Bank 0/LED_{3}: track 23.9 -> 73.8 mm
- net /Button Bank 0/LED_{5}: track 116.1 -> 164.9 mm
- net /Button Bank 1/LED_{1}: track 178.1 -> 226.2 mm
- net /Button Bank 1/LED_{5}: track 234.1 -> 281.2 mm
- net VCC: track 449.6 -> 496.3 mm
- net /Button Bank 1/SW_{7}: track 249.7 -> 294.8 mm
- net /Button Bank 1/LED_{7}: track 209.2 -> 254.2 mm
- net /Button Bank 1/LED_{3}: track 143.6 -> 188.6 mm
- net /Button Bank 0/LED_{7}: track 91.9 -> 136.9 mm
- net /Button Bank 0/SW_{3}: track 70.5 -> 115.4 mm
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
Commit message: Rough outline of single row
Parts:
- removed the R18 at (355.1, 90.7)
- added R3: 47Ω, Resistor_SMD:R_0402_1005Metric, F.Cu at (137.7, 86.7)
- R1, R2: value 400R -> 1.6kΩ; footprint Resistor_THT:R_Axial_DIN0204_L3.6mm_D1.6mm_P5.08mm_Horizontal -> Resistor_SMD:R_0402_1005Metric
- R10, R11, R12, R13, R14, R15, R16, R17, R4, R5, R6, R7, R8, R9: value 47R -> 47Ω; footprint Resistor_THT:R_Axial_DIN0204_L3.6mm_D1.6mm_P5.08mm_Horizontal -> Resistor_SMD:R_0402_1005Metric
- R18: renamed from R3; value 47R -> 47Ω; footprint Resistor_THT:R_Axial_DIN0204_L3.6mm_D1.6mm_P5.08mm_Horizontal -> Resistor_SMD:R_0402_1005Metric
- U1, U2, U3, U4: footprint Package_DIP:DIP-16_W7.62mm -> Package_SO:SOIC-16_3.9x9.9mm_P1.27mm
- moved R18 225.8 mm to (356.0, 90.2)
- moved SW16 225.0 mm to (355.8, 81.0)
- moved U3 29.8 mm to (95.2, 87.0), turned to 0 degrees
- moved U1 29.6 mm to (95.2, 76.5), turned to 0 degrees
- moved J1 22.6 mm to (81.9, 71.7)
- moved J2 22.6 mm to (78.1, 71.6)
- moved R7 22.6 mm to (197.6, 86.7), turned to -90 degrees
- moved R1 22.4 mm to (115.0, 73.3), turned to 0 degrees
- moved R2 22.3 mm to (115.0, 83.7), turned to 0 degrees
- moved U2 15.3 mm to (110.3, 76.5), turned to 0 degrees
- moved U4 15.2 mm to (110.3, 87.0), turned to 0 degrees
- moved SW9 15.0 mm to (250.8, 81.0)
- moved SW1 15.0 mm to (130.8, 81.0)
- moved SW10 15.0 mm to (265.8, 81.0)
- moved SW11 15.0 mm to (280.8, 81.0)
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- renumbered SW0 to SW16
Connections:
- R18 pad 1: /Button Bank 0/SW_{0} -> /Button Bank 1/SW_{7}
- R6 pad 1: /Button Bank 0/SW_{4} -> /Button Bank 0/SW_{3}
- R7 pad 1: /Button Bank 0/SW_{3} -> /Button Bank 0/SW_{4}
- SW1 pad 2: /Button Bank 0/SW_{1} -> /Button Bank 0/SW_{0}
- SW1 pad 6: /Button Bank 0/LED_{1} -> /Button Bank 0/LED_{0}
- SW10 pad 2: /Button Bank 1/SW_{2} -> /Button Bank 1/SW_{1}
- SW10 pad 6: /Button Bank 1/LED_{2} -> /Button Bank 1/LED_{1}
- SW11 pad 2: /Button Bank 1/SW_{3} -> /Button Bank 1/SW_{2}
- SW11 pad 6: /Button Bank 1/LED_{3} -> /Button Bank 1/LED_{2}
- SW12 pad 2: /Button Bank 1/SW_{4} -> /Button Bank 1/SW_{3}
- SW12 pad 6: /Button Bank 1/LED_{4} -> /Button Bank 1/LED_{3}
- SW13 pad 2: /Button Bank 1/SW_{5} -> /Button Bank 1/SW_{4}
- SW13 pad 6: /Button Bank 1/LED_{5} -> /Button Bank 1/LED_{4}
- SW14 pad 2: /Button Bank 1/SW_{6} -> /Button Bank 1/SW_{5}
- SW14 pad 6: /Button Bank 1/LED_{6} -> /Button Bank 1/LED_{5}
- SW15 pad 2: /Button Bank 1/SW_{7} -> /Button Bank 1/SW_{6}
- SW15 pad 6: /Button Bank 1/LED_{7} -> /Button Bank 1/LED_{6}
- SW16 pad 2: /Button Bank 0/SW_{0} -> /Button Bank 1/SW_{7}
- SW16 pad 6: /Button Bank 0/LED_{0} -> /Button Bank 1/LED_{7}
- SW2 pad 2: /Button Bank 0/SW_{2} -> /Button Bank 0/SW_{1}
- SW2 pad 6: /Button Bank 0/LED_{2} -> /Button Bank 0/LED_{1}
- SW3 pad 2: /Button Bank 0/SW_{3} -> /Button Bank 0/SW_{2}
- SW3 pad 6: /Button Bank 0/LED_{3} -> /Button Bank 0/LED_{2}
- SW4 pad 2: /Button Bank 0/SW_{4} -> /Button Bank 0/SW_{3}
- SW4 pad 6: /Button Bank 0/LED_{4} -> /Button Bank 0/LED_{3}
- SW5 pad 2: /Button Bank 0/SW_{5} -> /Button Bank 0/SW_{4}
- SW5 pad 6: /Button Bank 0/LED_{5} -> /Button Bank 0/LED_{4}
- SW6 pad 2: /Button Bank 0/SW_{6} -> /Button Bank 0/SW_{5}
- SW6 pad 6: /Button Bank 0/LED_{6} -> /Button Bank 0/LED_{5}
- SW7 pad 2: /Button Bank 0/SW_{7} -> /Button Bank 0/SW_{6}
- SW7 pad 6: /Button Bank 0/LED_{7} -> /Button Bank 0/LED_{6}
- SW8 pad 2: /Button Bank 1/SW_{0} -> /Button Bank 0/SW_{7}
- SW8 pad 6: /Button Bank 1/LED_{0} -> /Button Bank 0/LED_{7}
- SW9 pad 2: /Button Bank 1/SW_{1} -> /Button Bank 1/SW_{0}
- SW9 pad 6: /Button Bank 1/LED_{1} -> /Button Bank 1/LED_{0}
- U2 pad 10: /Button Bank 1/LED_{5} -> /Button Bank 0/LED_{5}
- U2 pad 11: /Button Bank 1/LED_{6} -> /Button Bank 0/LED_{6}
- U2 pad 12: /Button Bank 1/LED_{7} -> /Button Bank 0/LED_{7}
- U2 pad 14: /DO_{LED} -> /Button Bank 0/DO_{LED}
- U2 pad 2: /Button Bank 0/DO_{LED} -> /DI_{LED}
- U2 pad 5: /Button Bank 1/LED_{0} -> /Button Bank 0/LED_{0}
- U2 pad 6: /Button Bank 1/LED_{1} -> /Button Bank 0/LED_{1}
- U2 pad 7: /Button Bank 1/LED_{2} -> /Button Bank 0/LED_{2}
- U2 pad 8: /Button Bank 1/LED_{3} -> /Button Bank 0/LED_{3}
- U2 pad 9: /Button Bank 1/LED_{4} -> /Button Bank 0/LED_{4}
- U4 pad 10: /Button Bank 0/LED_{5} -> /Button Bank 1/LED_{5}
- U4 pad 11: /Button Bank 0/LED_{6} -> /Button Bank 1/LED_{6}
- U4 pad 12: /Button Bank 0/LED_{7} -> /Button Bank 1/LED_{7}
- U4 pad 14: /Button Bank 0/DO_{LED} -> /DO_{LED}
- U4 pad 2: /DI_{LED} -> /Button Bank 0/DO_{LED}
- U4 pad 5: /Button Bank 0/LED_{0} -> /Button Bank 1/LED_{0}
- U4 pad 6: /Button Bank 0/LED_{1} -> /Button Bank 1/LED_{1}
- U4 pad 7: /Button Bank 0/LED_{2} -> /Button Bank 1/LED_{2}
- U4 pad 8: /Button Bank 0/LED_{3} -> /Button Bank 1/LED_{3}
- U4 pad 9: /Button Bank 0/LED_{4} -> /Button Bank 1/LED_{4}
Routing:
- net /Button Bank 0/SW_{1}: track 165.0 -> 70.0 mm, vias 0 -> 1
- net /Button Bank 1/SW_{0}: track 253.7 -> 164.9 mm
- net /Button Bank 0/SW_{0}: track 137.6 -> 55.6 mm, vias 0 -> 1
- net /Button Bank 1/SW_{5}: track 331.4 -> 251.8 mm
- net /Button Bank 0/SW_{4}: track 203.6 -> 125.7 mm, vias 0 -> 1
- net /Button Bank 0/SW_{5}: track 217.7 -> 143.1 mm, vias 0 -> 1
- net /Button Bank 0/LED_{0}: track 97.3 -> 23.0 mm, vias 0 -> 1
- net /Button Bank 0/LED_{1}: track 109.9 -> 37.8 mm, vias 0 -> 1
- net /Button Bank 0/LED_{5}: track 164.9 -> 96.2 mm
- net /Button Bank 1/SW_{4}: track 300.7 -> 234.0 mm
- net /Button Bank 0/LED_{4}: track 147.1 -> 81.3 mm
- net /Button Bank 1/LED_{5}: track 281.2 -> 218.2 mm, vias 0 -> 1
- net LE_{LED}: track 70.8 -> 16.8 mm
- net /Button Bank 1/LED_{0}: track 214.0 -> 161.0 mm, vias 0 -> 1
- net GND: track 0.00 -> 51.8 mm, vias 0 -> 22
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
Commit message: 3 rows of 16 buttons; SMT
Parts:
- added R19: 1.6kΩ, Resistor_SMD:R_0402_1005Metric, F.Cu at (76.4, 92.1)
- added R20: 1.6kΩ, Resistor_SMD:R_0402_1005Metric, F.Cu at (76.4, 102.5)
- added R21: 47Ω, Resistor_SMD:R_0402_1005Metric, F.Cu at (99.0, 105.4)
- added R22: 47Ω, Resistor_SMD:R_0402_1005Metric, F.Cu at (113.9, 105.4)
- added R23: 47Ω, Resistor_SMD:R_0402_1005Metric, F.Cu at (129.2, 105.4)
- added R24: 47Ω, Resistor_SMD:R_0402_1005Metric, F.Cu at (144.0, 105.3)
- added R25: 47Ω, Resistor_SMD:R_0402_1005Metric, F.Cu at (158.9, 105.4)
- added R26: 47Ω, Resistor_SMD:R_0402_1005Metric, F.Cu at (174.1, 105.4)
- added R27: 47Ω, Resistor_SMD:R_0402_1005Metric, F.Cu at (189.0, 105.4)
- added R28: 47Ω, Resistor_SMD:R_0402_1005Metric, F.Cu at (204.0, 105.4)
- added R29: 47Ω, Resistor_SMD:R_0402_1005Metric, F.Cu at (219.0, 105.4)
- added R30: 47Ω, Resistor_SMD:R_0402_1005Metric, F.Cu at (234.0, 105.4)
- added R31: 47Ω, Resistor_SMD:R_0402_1005Metric, F.Cu at (249.0, 105.4)
- added R32: 47Ω, Resistor_SMD:R_0402_1005Metric, F.Cu at (264.0, 105.4)
- added R33: 47Ω, Resistor_SMD:R_0402_1005Metric, F.Cu at (279.1, 105.4)
- added R34: 47Ω, Resistor_SMD:R_0402_1005Metric, F.Cu at (293.9, 105.4)
- added R35: 47Ω, Resistor_SMD:R_0402_1005Metric, F.Cu at (309.1, 105.4)
- added R36: 47Ω, Resistor_SMD:R_0402_1005Metric, F.Cu at (317.4, 109.0)
- added R37: 1.6kΩ, Resistor_SMD:R_0402_1005Metric, F.Cu at (76.4, 119.0)
- added R38: 1.6kΩ, Resistor_SMD:R_0402_1005Metric, F.Cu at (76.4, 129.4)
- added R39: 47Ω, Resistor_SMD:R_0402_1005Metric, F.Cu at (99.0, 132.3)
- added R40: 47Ω, Resistor_SMD:R_0402_1005Metric, F.Cu at (113.9, 132.3)
- added R41: 47Ω, Resistor_SMD:R_0402_1005Metric, F.Cu at (129.2, 132.3)
- added R42: 47Ω, Resistor_SMD:R_0402_1005Metric, F.Cu at (144.0, 132.2)
- added R43: 47Ω, Resistor_SMD:R_0402_1005Metric, F.Cu at (158.9, 132.3)
- added R44: 47Ω, Resistor_SMD:R_0402_1005Metric, F.Cu at (174.1, 132.3)
- added R45: 47Ω, Resistor_SMD:R_0402_1005Metric, F.Cu at (189.0, 132.3)
- added R46: 47Ω, Resistor_SMD:R_0402_1005Metric, F.Cu at (204.0, 132.3)
- added R47: 47Ω, Resistor_SMD:R_0402_1005Metric, F.Cu at (219.0, 132.3)
- added R48: 47Ω, Resistor_SMD:R_0402_1005Metric, F.Cu at (234.0, 132.3)
- added R49: 47Ω, Resistor_SMD:R_0402_1005Metric, F.Cu at (249.0, 132.3)
- added R50: 47Ω, Resistor_SMD:R_0402_1005Metric, F.Cu at (264.0, 132.3)
- added R51: 47Ω, Resistor_SMD:R_0402_1005Metric, F.Cu at (279.1, 132.3)
- added R52: 47Ω, Resistor_SMD:R_0402_1005Metric, F.Cu at (293.9, 132.3)
- added R53: 47Ω, Resistor_SMD:R_0402_1005Metric, F.Cu at (309.1, 132.3)
- added R54: 47Ω, Resistor_SMD:R_0402_1005Metric, F.Cu at (317.4, 135.9)
- added SW17: ~, Local:PB86, B.Cu at (92.2, 99.8)
- added SW18: ~, Local:PB86, B.Cu at (107.2, 99.8)
- added SW19: ~, Local:PB86, B.Cu at (122.2, 99.8)
- added SW20: ~, Local:PB86, B.Cu at (137.2, 99.8)
- added SW21: ~, Local:PB86, B.Cu at (152.2, 99.8)
- added SW22: ~, Local:PB86, B.Cu at (167.2, 99.8)
- added SW23: ~, Local:PB86, B.Cu at (182.2, 99.8)
- added SW24: ~, Local:PB86, B.Cu at (197.2, 99.8)
- added SW25: ~, Local:PB86, B.Cu at (212.2, 99.8)
- added SW26: ~, Local:PB86, B.Cu at (227.2, 99.8)
- added SW27: ~, Local:PB86, B.Cu at (242.2, 99.8)
- added SW28: ~, Local:PB86, B.Cu at (257.2, 99.8)
- added SW29: ~, Local:PB86, B.Cu at (272.2, 99.8)
- added SW30: ~, Local:PB86, B.Cu at (287.2, 99.8)
- added SW31: ~, Local:PB86, B.Cu at (302.2, 99.8)
- added SW32: ~, Local:PB86, B.Cu at (317.2, 99.8)
- added SW33: ~, Local:PB86, B.Cu at (92.2, 126.7)
- added SW34: ~, Local:PB86, B.Cu at (107.2, 126.7)
- added SW35: ~, Local:PB86, B.Cu at (122.2, 126.7)
- added SW36: ~, Local:PB86, B.Cu at (137.2, 126.7)
- added SW37: ~, Local:PB86, B.Cu at (152.2, 126.7)
- added SW38: ~, Local:PB86, B.Cu at (167.2, 126.7)
- added SW39: ~, Local:PB86, B.Cu at (182.2, 126.7)
- added SW40: ~, Local:PB86, B.Cu at (197.2, 126.7)
- added SW41: ~, Local:PB86, B.Cu at (212.2, 126.7)
- added SW42: ~, Local:PB86, B.Cu at (227.2, 126.7)
- added SW43: ~, Local:PB86, B.Cu at (242.2, 126.7)
- added SW44: ~, Local:PB86, B.Cu at (257.2, 126.7)
- added SW45: ~, Local:PB86, B.Cu at (272.2, 126.7)
- added SW46: ~, Local:PB86, B.Cu at (287.2, 126.7)
- added SW47: ~, Local:PB86, B.Cu at (302.2, 126.7)
- added SW48: ~, Local:PB86, B.Cu at (317.2, 126.7)
- added U10: 74HC165, Package_SO:SOIC-16_3.9x9.9mm_P1.27mm, F.Cu at (56.6, 132.7)
- added U11: TLC5916, Package_SO:SOIC-16_3.9x9.9mm_P1.27mm, F.Cu at (71.6, 122.2)
- added U12: TLC5916, Package_SO:SOIC-16_3.9x9.9mm_P1.27mm, F.Cu at (71.6, 132.7)
- added U5: 74HC165, Package_SO:SOIC-16_3.9x9.9mm_P1.27mm, F.Cu at (56.6, 95.2)
- added U6: 74HC165, Package_SO:SOIC-16_3.9x9.9mm_P1.27mm, F.Cu at (56.6, 105.8)
- added U7: TLC5916, Package_SO:SOIC-16_3.9x9.9mm_P1.27mm, F.Cu at (71.6, 95.2)
- added U8: TLC5916, Package_SO:SOIC-16_3.9x9.9mm_P1.27mm, F.Cu at (71.6, 105.8)
- added U9: 74HC165, Package_SO:SOIC-16_3.9x9.9mm_P1.27mm, F.Cu at (56.6, 122.2)
- moved H2 103.1 mm to (38.5, 138.2)
- moved H1 85.9 mm to (38.5, 61.9)
- moved H4 64.3 mm to (327.9, 138.2)
- moved J2 56.2 mm to (43.8, 116.2)
- moved H3 40.3 mm to (327.9, 61.9)
- moved SW10 39.5 mm to (227.2, 72.8)
- moved SW11 39.5 mm to (242.2, 72.8)
- moved R10 39.5 mm to (204.0, 78.5)
- moved R11 39.5 mm to (219.0, 78.5)
- moved R16 39.5 mm to (293.9, 78.5)
- moved R17 39.5 mm to (309.1, 78.5)
- moved R7 39.5 mm to (158.9, 78.5)
- moved R8 39.5 mm to (174.1, 78.5)
- moved SW12 39.5 mm to (257.2, 72.8)
- moved SW13 39.5 mm to (272.2, 72.8)
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Connections:
- U3 pad 10: /DI_{SW} -> /Button Bank 1/DI_{SW}
- U4 pad 14: /DO_{LED} -> /Button Bank 1/DO_{LED}
Routing:
- net GND: track 51.8 -> 2487.0 mm, vias 22 -> 72
- net VCC: track 453.3 -> 1520.8 mm
- net /Button Bank 5/LED_{4}: track 0.00 -> 299.5 mm, vias 0 -> 1
- net /Button Bank 3/LED_{4}: track 0.00 -> 299.5 mm, vias 0 -> 1
- net /Button Bank 5/SW_{7}: track 0.00 -> 283.5 mm
- net /Button Bank 3/SW_{7}: track 0.00 -> 283.5 mm
- net /Button Bank 5/SW_{6}: track 0.00 -> 269.2 mm
- net /Button Bank 3/SW_{6}: track 0.00 -> 269.2 mm
- net /Button Bank 5/SW_{5}: track 0.00 -> 251.8 mm
- net /Button Bank 3/SW_{5}: track 0.00 -> 251.8 mm
- net /Button Bank 5/LED_{7}: track 0.00 -> 247.9 mm, vias 0 -> 1
- net /Button Bank 3/LED_{7}: track 0.00 -> 247.9 mm, vias 0 -> 1
- net /Button Bank 5/SW_{4}: track 0.00 -> 234.0 mm
- net /Button Bank 3/SW_{4}: track 0.00 -> 234.0 mm
- net /Button Bank 5/LED_{6}: track 0.00 -> 233.1 mm, vias 0 -> 1
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Other:
- board size 316.6 x 28.5 mm -> 296.2 x 83.2 mm
- board text removed: "3V3"
- board text removed: "CHAIN"
- board text removed: "CLK"
- board text removed: "DATA"
- board text removed: "GND"
- board text removed: "LCH"
- board text removed: "LED"
- board text removed: "MCU"
- board text removed: "SWITCH"
- board text removed: "~{LCH}"
- board text removed: "~{OE}"

Commit message: Revert "3 rows of 16 buttons; SMT"
This reverts commit c08e4dc0c350e57a2ca7329c2459be699e742724.
Parts:
- removed R19, R20, R37, R38: 1.6kΩ, Resistor_SMD:R_0402_1005Metric
- removed R21, R22, R23, R24, R25, R26, R27, R28, R29, R30, R31, R32, R33, R34, R35, R36, R39, R40, R41, R42, R43, R44, R45, R46, R47, R48, R49, R50, R51, R52, R53, R54: 47Ω, Resistor_SMD:R_0402_1005Metric
- removed SW17, SW18, SW19, SW20, SW21, SW22, SW23, SW24, SW25, SW26, SW27, SW28, SW29, SW30, SW31, SW32, SW33, SW34, SW35, SW36, SW37, SW38, SW39, SW40, SW41, SW42, SW43, SW44, SW45, SW46, SW47, SW48: ~, Local:PB86
- removed U10, U5, U6, U9: 74HC165, Package_SO:SOIC-16_3.9x9.9mm_P1.27mm
- removed U11, U12, U7, U8: TLC5916, Package_SO:SOIC-16_3.9x9.9mm_P1.27mm
- moved H2 103.1 mm to (120.7, 76.1)
- moved H1 85.9 mm to (120.7, 86.7)
- moved H4 64.3 mm to (365.6, 86.1)
- moved J2 56.2 mm to (78.1, 71.6)
- moved H3 40.3 mm to (365.6, 76.0)
- moved SW10 39.5 mm to (265.8, 81.0)
- moved SW11 39.5 mm to (280.8, 81.0)
- moved R10 39.5 mm to (242.7, 86.7)
- moved R11 39.5 mm to (257.7, 86.7)
- moved R16 39.5 mm to (332.6, 86.7)
- moved R17 39.5 mm to (347.7, 86.7)
- moved R7 39.5 mm to (197.6, 86.7)
- moved R8 39.5 mm to (212.7, 86.7)
- moved SW12 39.5 mm to (295.8, 81.0)
- moved SW13 39.5 mm to (310.8, 81.0)
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Connections:
- U3 pad 10: /Button Bank 1/DI_{SW} -> /DI_{SW}
- U4 pad 14: /Button Bank 1/DO_{LED} -> /DO_{LED}
Routing:
- net GND: track 2487.0 -> 51.8 mm, vias 72 -> 22
- net VCC: track 1520.8 -> 453.3 mm
- net /Button Bank 5/LED_{4}: track 299.5 -> 0.00 mm, vias 1 -> 0
- net /Button Bank 3/LED_{4}: track 299.5 -> 0.00 mm, vias 1 -> 0
- net /Button Bank 5/SW_{7}: track 283.5 -> 0.00 mm
- net /Button Bank 3/SW_{7}: track 283.5 -> 0.00 mm
- net /Button Bank 5/SW_{6}: track 269.2 -> 0.00 mm
- net /Button Bank 3/SW_{6}: track 269.2 -> 0.00 mm
- net /Button Bank 5/SW_{5}: track 251.8 -> 0.00 mm
- net /Button Bank 3/SW_{5}: track 251.8 -> 0.00 mm
- net /Button Bank 5/LED_{7}: track 247.9 -> 0.00 mm, vias 1 -> 0
- net /Button Bank 3/LED_{7}: track 247.9 -> 0.00 mm, vias 1 -> 0
- net /Button Bank 5/SW_{4}: track 234.0 -> 0.00 mm
- net /Button Bank 3/SW_{4}: track 234.0 -> 0.00 mm
- net /Button Bank 5/LED_{6}: track 233.1 -> 0.00 mm, vias 1 -> 0
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Other:
- board size 296.2 x 83.2 mm -> 316.6 x 28.5 mm
- board text added: "3V3"
- board text added: "CHAIN"
- board text added: "CLK"
- board text added: "DATA"
- board text added: "GND"
- board text added: "LCH"
- board text added: "LED"
- board text added: "MCU"
- board text added: "SWITCH"
- board text added: "~{LCH}"
- board text added: "~{OE}"

Commit message: Rework single row to use more of the vertical space between button contacts.
Parts:
- removed H1, H2, H3, H4: MountingHole, MountingHole:MountingHole_3.2mm_M3
- removed J1: Output, Connector_PinHeader_2.54mm:PinHeader_1x09_P2.54mm_Vertical
- removed J2: Input, Connector_PinHeader_2.54mm:PinHeader_1x09_P2.54mm_Vertical
- moved U1 21.7 mm to (113.4, 88.3), turned to 90 degrees
- moved U4 14.5 mm to (99.8, 77.0), turned to -90 degrees
- moved R2 10.5 mm to (105.5, 79.3), turned to -90 degrees
- moved R1 8.10 mm to (117.0, 81.2)
- moved U3 4.88 mm to (99.9, 88.3), turned to 90 degrees
- moved U2 3.03 mm to (113.3, 77.0), turned to -90 degrees
Routing:
- net GND: track 51.8 -> 135.9 mm, vias 22 -> 9
- net /Button Bank 1/LED_{4}: track 297.7 -> 221.9 mm, vias 1 -> 3
- net VCC: track 453.3 -> 400.2 mm, vias 0 -> 3
- net /Button Bank 0/SW_{6}: track 160.5 -> 118.0 mm, vias 1 -> 0
- net /Button Bank 0/SW_{7}: track 177.5 -> 135.4 mm, vias 1 -> 0
- net /DO_{LED}: track 52.4 -> 10.3 mm, vias 0 -> 1
- net /Button Bank 0/SW_{5}: track 143.1 -> 101.4 mm, vias 1 -> 0
- net /Button Bank 0/SW_{4}: track 125.7 -> 86.4 mm, vias 1 -> 0
- net /DI_{SW}: track 48.7 -> 11.2 mm, vias 0 -> 1
- net ~{OE_{LED}}: track 64.5 -> 35.0 mm, vias 0 -> 1
- net /Button Bank 0/SW_{3}: track 98.7 -> 72.2 mm, vias 1 -> 0
- net /DO_{SW}: track 0.00 -> 26.2 mm, vias 0 -> 1
- net /Button Bank 0/SW_{2}: track 84.6 -> 58.8 mm, vias 1 -> 0
- net /Button Bank 0/SW_{1}: track 70.0 -> 44.4 mm, vias 1 -> 0
- net /Button Bank 0/SW_{0}: track 55.6 -> 30.1 mm, vias 1 -> 0
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- added copper zone on F.Cu, net GND
Other:
- board outline removed
- board text removed: "3V3"
- board text removed: "CHAIN"
- board text removed: "CLK"
- board text removed: "DATA"
- board text removed: "GND"
- board text removed: "LCH"
- board text removed: "LED"
- board text removed: "MCU"
- board text removed: "SWITCH"
- board text removed: "~{LCH}"
- board text removed: "~{OE}"
