File: KiCAD/DrumKitButtons.kicad_pcb (KiCad board)
At the start: 2 copper layers, 297.2 x 76.2 mm, 125 parts, among them J1 Output, J2 Input, U1 74HC165, U10 74HC165, U11 TLC5916, U12 TLC5916, U2 TLC5916, U3 74HC165, U4 TLC5916, U5 74HC165, U6 74HC165, U7 TLC5916, U8 TLC5916, U9 74HC165

Commit message: DNP for headers; switch 5916->5917
Parts:
- U11, U12, U2, U4, U7, U8: value TLC5916 -> TLC5917QDRQ1
Connections:
- R10 pad 1: /Button Bank 0/SW_{7} -> GND
- R10 pad 2: GND -> /Button Bank 0/SW_{7}
- R11 pad 1: /Button Bank 1/SW_{0} -> GND
- R11 pad 2: GND -> /Button Bank 1/SW_{0}
- R12 pad 1: /Button Bank 1/SW_{1} -> GND
- R12 pad 2: GND -> /Button Bank 1/SW_{1}
- R13 pad 1: /Button Bank 1/SW_{2} -> GND
- R13 pad 2: GND -> /Button Bank 1/SW_{2}
- R14 pad 1: /Button Bank 1/SW_{3} -> GND
- R14 pad 2: GND -> /Button Bank 1/SW_{3}
- R15 pad 1: /Button Bank 1/SW_{4} -> GND
- R15 pad 2: GND -> /Button Bank 1/SW_{4}
- R16 pad 1: /Button Bank 1/SW_{5} -> GND
- R16 pad 2: GND -> /Button Bank 1/SW_{5}
- R17 pad 1: /Button Bank 1/SW_{6} -> GND
- R17 pad 2: GND -> /Button Bank 1/SW_{6}
- R18 pad 1: /Button Bank 1/SW_{7} -> GND
- R18 pad 2: GND -> /Button Bank 1/SW_{7}
- R21 pad 1: /Button Bank 2/SW_{0} -> GND
- R21 pad 2: GND -> /Button Bank 2/SW_{1}
- R22 pad 1: /Button Bank 2/SW_{1} -> GND
- R22 pad 2: GND -> /Button Bank 2/SW_{0}
- R23 pad 1: /Button Bank 2/SW_{2} -> GND
- R23 pad 2: GND -> /Button Bank 2/SW_{4}
- R24 pad 1: /Button Bank 2/SW_{3} -> GND
- R24 pad 2: GND -> /Button Bank 2/SW_{7}
- R25 pad 1: /Button Bank 2/SW_{4} -> GND
- R25 pad 2: GND -> /Button Bank 2/SW_{3}
- R26 pad 1: /Button Bank 2/SW_{5} -> GND
- R26 pad 2: GND -> /Button Bank 2/SW_{6}
- R27 pad 1: /Button Bank 2/SW_{6} -> GND
- R27 pad 2: GND -> /Button Bank 2/SW_{2}
- R28 pad 1: /Button Bank 2/SW_{7} -> GND
- R28 pad 2: GND -> /Button Bank 2/SW_{5}
- R29 pad 1: /Button Bank 3/SW_{0} -> GND
- R29 pad 2: GND -> /Button Bank 3/SW_{1}
- R3 pad 1: /Button Bank 0/SW_{0} -> GND
- R3 pad 2: GND -> /Button Bank 0/SW_{0}
- R30 pad 1: /Button Bank 3/SW_{1} -> GND
- R30 pad 2: GND -> /Button Bank 3/SW_{0}
- R31 pad 1: /Button Bank 3/SW_{2} -> GND
- R31 pad 2: GND -> /Button Bank 3/SW_{4}
- R32 pad 1: /Button Bank 3/SW_{3} -> GND
- R32 pad 2: GND -> /Button Bank 3/SW_{7}
- R33 pad 1: /Button Bank 3/SW_{4} -> GND
- R33 pad 2: GND -> /Button Bank 3/SW_{3}
- R34 pad 1: /Button Bank 3/SW_{5} -> GND
- R34 pad 2: GND -> /Button Bank 3/SW_{6}
- R35 pad 1: /Button Bank 3/SW_{6} -> GND
- R35 pad 2: GND -> /Button Bank 3/SW_{2}
- R36 pad 1: /Button Bank 3/SW_{7} -> GND
- R36 pad 2: GND -> /Button Bank 3/SW_{5}
- R39 pad 1: /Button Bank 4/SW_{0} -> GND
- R39 pad 2: GND -> /Button Bank 4/SW_{1}
- R4 pad 1: /Button Bank 0/SW_{1} -> GND
- R4 pad 2: GND -> /Button Bank 0/SW_{1}
- R40 pad 1: /Button Bank 4/SW_{1} -> GND
- R40 pad 2: GND -> /Button Bank 4/SW_{0}
- R41 pad 1: /Button Bank 4/SW_{2} -> GND
- R41 pad 2: GND -> /Button Bank 4/SW_{4}
- R42 pad 1: /Button Bank 4/SW_{3} -> GND
- R42 pad 2: GND -> /Button Bank 4/SW_{7}
- R43 pad 1: /Button Bank 4/SW_{4} -> GND
- R43 pad 2: GND -> /Button Bank 4/SW_{3}
- R44 pad 1: /Button Bank 4/SW_{5} -> GND
- R44 pad 2: GND -> /Button Bank 4/SW_{6}
- R45 pad 1: /Button Bank 4/SW_{6} -> GND
- R45 pad 2: GND -> /Button Bank 4/SW_{2}
- R46 pad 1: /Button Bank 4/SW_{7} -> GND
- R46 pad 2: GND -> /Button Bank 4/SW_{5}
- R47 pad 1: /Button Bank 5/SW_{0} -> GND
- R47 pad 2: GND -> /Button Bank 5/SW_{1}
- R48 pad 1: /Button Bank 5/SW_{1} -> GND
- R48 pad 2: GND -> /Button Bank 5/SW_{0}
- R49 pad 1: /Button Bank 5/SW_{2} -> GND
- R49 pad 2: GND -> /Button Bank 5/SW_{4}
- R5 pad 1: /Button Bank 0/SW_{2} -> GND
- R5 pad 2: GND -> /Button Bank 0/SW_{2}
- R50 pad 1: /Button Bank 5/SW_{3} -> GND
- R50 pad 2: GND -> /Button Bank 5/SW_{7}
- R51 pad 1: /Button Bank 5/SW_{4} -> GND
- R51 pad 2: GND -> /Button Bank 5/SW_{3}
- R52 pad 1: /Button Bank 5/SW_{5} -> GND
- R52 pad 2: GND -> /Button Bank 5/SW_{6}
- R53 pad 1: /Button Bank 5/SW_{6} -> GND
- R53 pad 2: GND -> /Button Bank 5/SW_{2}
- R54 pad 1: /Button Bank 5/SW_{7} -> GND
- R54 pad 2: GND -> /Button Bank 5/SW_{5}
- R6 pad 1: /Button Bank 0/SW_{3} -> GND
- R6 pad 2: GND -> /Button Bank 0/SW_{3}
- R7 pad 1: /Button Bank 0/SW_{4} -> GND
- R7 pad 2: GND -> /Button Bank 0/SW_{4}
- R8 pad 1: /Button Bank 0/SW_{5} -> GND
- R8 pad 2: GND -> /Button Bank 0/SW_{5}
- R9 pad 1: /Button Bank 0/SW_{6} -> GND
- R9 pad 2: GND -> /Button Bank 0/SW_{6}

Commit message: fix ERC/DRC violations
Parts:
- moved R28 60.1 mm to (242.7, 61.3), turned to 90 degrees
- moved R46 60.1 mm to (242.7, 86.7), turned to 90 degrees
- moved R29 60.1 mm to (287.6, 61.3), turned to 90 degrees
- moved R48 60.1 mm to (287.6, 86.7), turned to 90 degrees
- moved R22 59.8 mm to (167.9, 61.3), turned to 90 degrees
- moved R41 59.8 mm to (167.9, 86.7), turned to 90 degrees
- moved R52 53.5 mm to (356.0, 64.8), turned to 180 degrees
- moved R54 53.5 mm to (356.0, 90.2), turned to 180 degrees
- moved R33 30.1 mm to (317.7, 61.3), turned to 90 degrees
- moved R51 30.1 mm to (317.7, 86.7), turned to 90 degrees
- moved R25 30.0 mm to (212.7, 61.3), turned to 90 degrees
- moved R42 30.0 mm to (212.7, 86.7), turned to 90 degrees
- moved R24 29.7 mm to (197.6, 61.3), turned to 90 degrees
- moved R43 29.7 mm to (197.6, 86.7), turned to 90 degrees
- moved R32 23.7 mm to (332.6, 61.3), turned to 90 degrees
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- renumbered H3 to H4, H3 to H5, H3 to H6, H3 to H7, H3 to H8, H4 to H9, R2 to R1, R20 to R18, R3 to R2, R22 to R20, R27 to R22, R25 to R23, R23 to R24, R28 to R25, R30 to R27, R24 to R28, R35 to R29, R1 to R3, R29 to R30, R33 to R31, R36 to R32, R31 to R33, R18 to R35, R38 to R36, R40 to R38, R43 to R40, R45 to R41, R46 to R42, R41 to R43, R48 to R45, R42 to R46, R53 to R48, R51 to R49, R54 to R50, R49 to R51, R32 to R52, R52 to R53, R50 to R54, SW16 to SW1, SW7 to SW10, SW5 to SW11, SW6 to SW12, SW4 to SW13, SW3 to SW14, SW2 to SW15, SW1 to SW16, SW32 to SW17, SW30 to SW18, SW31 to SW19, SW15 to SW2, SW28 to SW20, SW29 to SW21, SW27 to SW22, SW26 to SW23, SW25 to SW24, SW23 to SW25, SW24 to SW26, SW21 to SW27, SW22 to SW28, SW20 to SW29, SW14 to SW3, SW19 to SW30, SW18 to SW31, SW17 to SW32, SW48 to SW33, SW46 to SW34, SW47 to SW35, SW45 to SW36, SW44 to SW37, SW43 to SW38, SW41 to SW39, SW12 to SW4, SW42 to SW40, SW40 to SW41, SW39 to SW42, SW38 to SW43, SW37 to SW44, SW36 to SW45, SW34 to SW46, SW35 to SW47, SW33 to SW48, SW13 to SW5, SW11 to SW6, SW10 to SW7, SW9 to SW8, SW8 to SW9, U4 to U1, U11 to U10, U12 to U11, U10 to U12, U1 to U2, U2 to U3, U3 to U4, U8 to U5, U5 to U7, U7 to U8
Connections:
- net /Button Bank 0/Net-(U4-R-EXT) renamed /Button Bank 0/R_{ext}
- net /Button Bank 1/Net-(U4-R-EXT) renamed /Button Bank 1/R_{ext}
- net /Button Bank 2/Net-(U4-R-EXT) renamed /Button Bank 2/R_{ext}
- net /Button Bank 3/Net-(U4-R-EXT) renamed /Button Bank 3/R_{ext}
- net /Button Bank 4/Net-(U4-R-EXT) renamed /Button Bank 4/R_{ext}
- net /Button Bank 5/Net-(U4-R-EXT) renamed /Button Bank 5/R_{ext}
Routing:
- net CLK_{LED}: track 171.9 -> 172.6 mm
- net /DO_{SW}: vias 1 -> 0
- net /DI_{LED}: vias 1 -> 0
- net /DO_{LED}: vias 1 -> 0
