File: KiCAD/DrumKitButtons.kicad_sch (KiCad schematic)
At the start: 6 parts, among them J1 Output, J2 Input

Commit message: DNP for headers; switch 5916->5917
Parts:
- J1, J2: now not fitted
Changed lines of the file:
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@@
 		(in_bom yes)
 		(on_board yes)
-		(dnp no)
+		(dnp yes)
 		(fields_autoplaced yes)
 		(property "Reference" "J1"
@@
 		(in_bom yes)
 		(on_board yes)
-		(dnp no)
+		(dnp yes)
 		(fields_autoplaced yes)
 		(property "Reference" "J2"

Commit message: fix ERC/DRC violations
Parts:
- added H3, H4, H5, H6, H7: MountingHole, MountingHole:MountingHole_3.2mm_M3, symbol Mechanical:MountingHole
- renumbered H3 to H8, H4 to H9
Other:
- moved on the sheet: H8, H9
